Commit message: Added Gazebo files

File: description/robot.urdf.xacro (robot description, xacro)
@@ -2,3 +2,4 @@
 <robot xmlns:xacro="http://www.ros.org/wiki/xacro"  name="holobot">
     <xacro:include filename="robot_core.xacro"/>
+    <!-- <xacro:include filename="robot_control.xacro"/> -->
 </robot>

File: description/robot_core.xacro (robot description, xacro)
@@ -39,4 +39,7 @@
         </xacro:inertial_box>
     </link>
+    <gazebo reference="chassis">
+        <material>Gazebo/White</material>
+    </gazebo>
     <joint name="front_left_wheel_joint" type="continuous">
         <parent link="base_link"/>
@@ -61,4 +64,7 @@
         </xacro:inertial_cylinder>
     </link>
+    <gazebo reference="front_left_wheel">
+        <material>Gazebo/Black</material>
+    </gazebo>
     <joint name="front_right_wheel_joint" type="continuous">
         <parent link="base_link"/>
@@ -83,4 +89,7 @@
         </xacro:inertial_cylinder>
     </link>
+    <gazebo reference="front_right_wheel">
+        <material>Gazebo/Black</material>
+    </gazebo>
     <joint name="back_left_wheel_joint" type="continuous">
         <parent link="base_link"/>
@@ -105,4 +114,7 @@
         </xacro:inertial_cylinder>
     </link>
+    <gazebo reference="back_left_wheel">
+        <material>Gazebo/Black</material>
+    </gazebo>
     <joint name="back_right_wheel_joint" type="continuous">
         <parent link="base_link"/>
@@ -127,3 +139,6 @@
         </xacro:inertial_cylinder>
     </link>
+    <gazebo reference="back_right_wheel">
+        <material>Gazebo/Black</material>
+    </gazebo>
 </robot>
